Commit message: now we can properly retarget motion to prestoe

File: protomotions/data/assets/urdf/prestoe_biped.urdf (robot description, URDF)
Before this commit: robot prestoe, 16 links, 15 joints
Links:
- added link head; visual sphere radius=0.0001
Joints:
- added joint head: type fixed, parent torso_link, child head, origin xyz=0 0 0.5 rpy=0 0 0
